Commit message: made review changes

File: my_robot/urdf/my_robot.xacro (robot description, xacro)
@@ -167,3 +167,15 @@
     <dynamics damping="1.0" friction="1.0" />
   </joint>
+<gazebo reference="chassis">
+  <material>Gazebo/Blue</material>
+</gazebo>
+<gazebo reference="camera">
+  <material>Gazebo/Red</material>
+</gazebo>
+<gazebo reference="left_front_wheel">
+  <material>Gazebo/Black</material>
+</gazebo>
+<gazebo reference="right_front_wheel">
+  <material>Gazebo/Black</material>
+</gazebo>
 </robot>
